Commit message: New URDF, launch files, README and beginning of orbslam configuration.

File: tcc_tello/description/urdf/tello.urdf.xacro (robot description, xacro)
@@ -12,19 +12,22 @@
       </inertial>
       <visual>
-        <origin xyz="0 0 0" rpy="0 0 ${90*pi/180}" />
+        <origin xyz="0 0 0" rpy="0 0 0" />
         <geometry>
-	  <mesh filename="package://tcc_tello/description/meshes/tello/tello.dae"/>
+	      <mesh filename="package://tcc_tello/description/meshes/tello/tello.dae"/>
         </geometry>
       </visual>
       <collision>
-        <origin xyz="0 0 0" rpy="0 0 ${90*pi/180}" />
+        <origin xyz="0 0 0" rpy="0 0 0" />
         <geometry>
-	  <mesh filename="package://tcc_tello/description/meshes/tello/tello.stl"/>
+	      <mesh filename="package://tcc_tello/description/meshes/tello/tello.dae"/>
         </geometry>
       </collision>
     </link>
+    <gazebo reference="base_link">
+        <material>Gazebo/White</material>
+    </gazebo>
     <!-- Sonar height sensor -->
-    <xacro:sonar_sensor name="sonar" parent="base_link" ros_topic="sonar_height" update_rate="10" min_range="0.03" max_range="3.0" field_of_view="${40*pi/180}" ray_count="3">
-      <origin xyz="0.0 -0.01 0.005" rpy="0 ${90*pi/180} ${90*pi/180}"/>
+    <xacro:sonar_sensor name="sonar" parent="base_link" ros_topic="sonar_height" update_rate="10" min_range="0.003" max_range="3.0" field_of_view="${40*pi/180}" ray_count="3">
+      <origin xyz="0.0 0.0 0.018" rpy="0 ${90*pi/180} 0"/>
     </xacro:sonar_sensor>
   </xacro:macro>

File: tcc_tello/description/urdf/tello_with_cam.gazebo.xacro (robot description, xacro)
@@ -1,5 +1,14 @@
 <?xml version="1.0"?>
 <robot name="quadrotor" xmlns:xacro="http://www.ros.org/wiki/xacro">
-    <xacro:include filename="$(find tcc_tello)/description/urdf/tello_with_cam.urdf.xacro" />
+    <xacro:property name="M_PI" value="3.1415926535897931" />
+    <!-- Included URDF Files -->
+    <xacro:include filename="$(find tcc_tello)/description/urdf/tello.urdf.xacro" />
+    <!-- Instantiate quadrotor_base_macro once (has no parameters atm) -->
+    <xacro:quadrotor_base_macro />
+    <!-- Forward facing camera -->
+    <xacro:include filename="$(find hector_sensors_description)/urdf/generic_camera.urdf.xacro" />
+    <xacro:generic_camera name="front_cam" parent="base_link" ros_topic="camera/image" cam_info_topic="camera/camera_info" update_rate="30" res_x="960" res_y="720" image_format="R8G8B8" hfov="90">
+      <origin xyz="0.048304 0 0.007574" rpy="0 0 0"/>
+    </xacro:generic_camera>
     <xacro:include filename="$(find hector_quadrotor_gazebo)/urdf/quadrotor_plugins.gazebo.xacro" />
 </robot>

Commit message: Add takeoff and land functions at gazebo_tello_control

File: tcc_tello/description/urdf/tello.urdf.xacro (robot description, xacro)
@@ -28,6 +28,6 @@
     </gazebo>
     <!-- Sonar height sensor -->
-    <xacro:sonar_sensor name="sonar" parent="base_link" ros_topic="sonar_height" update_rate="10" min_range="0.003" max_range="3.0" field_of_view="${40*pi/180}" ray_count="3">
-      <origin xyz="0.0 0.0 0.018" rpy="0 ${90*pi/180} 0"/>
+    <xacro:sonar_sensor name="sonar" parent="base_link" ros_topic="sonar_height" update_rate="10" min_range="0.02" max_range="3.0" field_of_view="${40*pi/180}" ray_count="3">
+      <origin xyz="0.0 0.0 0.02" rpy="0 ${90*pi/180} 0"/>
     </xacro:sonar_sensor>
   </xacro:macro>

Commit message: Configuração inicial tello orbslam simulação

File: tcc_tello/description/urdf/tello.urdf.xacro (robot description, xacro)
@@ -6,5 +6,5 @@
   <xacro:macro name="quadrotor_base_macro">
     <link name="base_link">
-      <inertial>
+     <inertial>
         <mass value="0.085" />
         <origin xyz="0 0 0" />
