Commit message: Atualização do nome do pacote

File: tello_pkg/description/urdf/generic_camera.urdf.xacro (robot description, xacro)
@@ -9,24 +9,4 @@
     </joint>
     <link name="${name}_link">
-<!--      <inertial>
-        <mass value="0.001" />
-        <origin xyz="0 0 0" rpy="0 0 0" />
-        <inertia ixx="0.0001" ixy="0" ixz="0" iyy="0.0001" iyz="0" izz="0.0001" />
-      </inertial>
-      <visual>
-        <origin xyz="0 0 0" rpy="0 0 0" />
-        <geometry>
-          <box size="0.01 0.01 0.01" />
-        </geometry>
-        <material name="Blue">
-          <color rgba="0.0 0.0 0.8 1"/>
-        </material>
-      </visual>
-      <collision>
-        <origin xyz="0 0 0" rpy="0 0 0" />
-        <geometry>
-          <box size="0.01 0.01 0.01" />
-        </geometry>
-      </collision>-->
     </link>
     <joint name="${name}_optical_joint" type="fixed">

File: tello_pkg/description/urdf/tello.urdf (robot description, URDF)
Before this commit: robot quadrotor, 4 links, 3 joints
Links:
- link base_link: geometry collision mesh filename=package://tello_pkg/description/meshes/tello/tello.dae; visual mesh filename=package://tello_pkg/description/meshes/tello/tello.dae

File: tello_pkg/description/urdf/tello.urdf.xacro (robot description, xacro)
@@ -14,5 +14,5 @@
         <origin xyz="0 0 0" rpy="0 0 0" />
         <geometry>
-	      <mesh filename="package://tcc_tello/description/meshes/tello/tello.dae"/>
+	      <mesh filename="package://tello_pkg/description/meshes/tello/tello.dae"/>
         </geometry>
       </visual>
@@ -20,5 +20,5 @@
         <origin xyz="0 0 0" rpy="0 0 0" />
         <geometry>
-	      <mesh filename="package://tcc_tello/description/meshes/tello/tello.dae"/>
+	      <mesh filename="package://tello_pkg/description/meshes/tello/tello.dae"/>
         </geometry>
       </collision>

File: tello_pkg/description/urdf/tello_with_cam.gazebo.xacro (robot description, xacro)
@@ -3,5 +3,5 @@
     <xacro:property name="M_PI" value="3.1415926535897931" />
     <!-- Included URDF Files -->
-    <xacro:include filename="$(find tcc_tello)/description/urdf/tello.urdf.xacro" />
+    <xacro:include filename="$(find tello_pkg)/description/urdf/tello.urdf.xacro" />
     <!-- Instantiate quadrotor_base_macro once (has no parameters atm) -->
     <xacro:quadrotor_base_macro />
